File: modules_lpc1115/smokedetector/Rauchmelder.sch (EAGLE design)
At the start: 75 parts, among them IC1 BD9G101, IC2 LPC1115, Q1 BC856, Q3 BCP52, Q4 ASFL, T1 BC847C, T2 BC817

Commit message: [RM] - rearranged diodes; added holes for pull out zip tie
Parts:
- C20: value 100n -> 100nF
- R8: value 5R6 -> 5R6 1210
Other:
- note added: "3.8.4"
- note removed: "3.8.3"
- moved on the sheet: C100, C104, C105, R6, R8
