File: misc/dap_debugger/SelfBus DAP Debugger.brd (EAGLE design)
At the start: 35.1 x 85.1 mm, 60 parts, among them CON1 MICRO-B_U254-051N-4BH806, CON2 SHF-105-01-X-D-TH, CON3 SHF-105-01-X-D-TH, CON4 SAMTEC-LTMM-105-02-T-D, IC1 74LVC1T45GW, IC2 74LVC2G07GV, IC3 74LVC2T45DC, IC4 74LVC2T45DC, SW1 BOOT, SW2 RESET, SW3 XKB7070-Z, U1 STM32F042FX, U2 AP2112K-3.3TRG1, U3 AP2331TDW

Commit message: [SB-DAP] - changed values to standard values
Parts:
- C18: value 10µF -> 10uF
- C3, C4, C5: value 4,7µF -> 4.7uF
Changed lines of the file:
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@@
 <drawing>
 <settings>
-<setting alwaysvectorfont="yes"/>
+<setting alwaysvectorfont="no"/>
 <setting verticaltext="up"/>
 </settings>
@@
 </layers>
 <board>
-<fusionsync huburn="a.YnVzaW5lc3M6dG9ubGluZTE5NDA" projecturn="a.YnVzaW5lc3M6dG9ubGluZTE5NDAjRDIwMTkxMTA3MjM1NzAyODUx" f3durn="urn:adsk.wipprod:dm.lineage:r5j3DoLdQL6_27IBNw_zwA" pcbguid="" lastpulledtime="" lastsyncedchangeguid="" latestrevisionid="5ee4731d-589f-44e8-8e76-53e9234253aa" lastsyncedrevisionid="5ee4731d-589f-44e8-8e76-53e9234253aa" lastboardhashguid="15e6d303-7afb-03e8-1037-e26f4ed606de" lastpushedtime="2021-06-07T18:27:28Z" linktopcb3d="true"/>
+<fusionsync huburn="a.YnVzaW5lc3M6dG9ubGluZTE5NDA" projecturn="a.YnVzaW5lc3M6dG9ubGluZTE5NDAjRDIwMTkxMTA3MjM1NzAyODUx" f3durn="urn:adsk.wipprod:dm.lineage:r5j3DoLdQL6_27IBNw_zwA" pcbguid="" lastpulledtime="" lastsyncedchangeguid="" latestrevisionid="5ee4731d-589f-44e8-8e76-53e9234253aa" lastsyncedrevisionid="5ee4731d-589f-44e8-8e76-53e9234253aa" lastboardhashguid="15e6d303-7afb-03e8-1037-e26f4ed606de" lastpushedtime="2021-06-07T18:27:28Z" linktopcb3d="false"/>
 <plain>
 <circle x="28.385" y="13.885" radius="1.25" width="0.1524" layer="20"/>
@@
 <attribute name="VALUE" x="9.963" y="13.462" size="1.016" layer="27" rot="R90" align="top-center"/>
 </element>
-<element name="C3" library="MyRCL" package="C0805" package3d_urn="urn:adsk.eagle:package:23617/2" value="4,7µF" x="12.065" y="15.494" smashed="yes">
+<element name="C3" library="MyRCL" package="C0805" package3d_urn="urn:adsk.eagle:package:23617/2" value="4.7uF" x="12.065" y="15.494" smashed="yes">
 <attribute name="NAME" x="12.065" y="16.791" size="1.016" layer="25" align="bottom-center"/>
 <attribute name="SPICEPREFIX" value="C" x="73.025" y="-37.846" size="1.778" layer="27" display="off"/>
 <attribute name="VALUE" x="13.265" y="15.875" size="1.016" layer="27" rot="R90" align="top-center"/>
 </element>
-<element name="C4" library="MyRCL" package="C0805" package3d_urn="urn:adsk.eagle:package:23617/2" value="4,7µF" x="9.906" y="26.543" smashed="yes">
+<element name="C4" library="MyRCL" package="C0805" package3d_urn="urn:adsk.eagle:package:23617/2" value="4.7uF" x="9.906" y="26.543" smashed="yes">
 <attribute name="NAME" x="12.673" y="26.543" size="1.016" layer="25" rot="R90" align="bottom-center"/>
 <attribute name="SPICEPREFIX" value="C" x="75.946" y="-26.797" size="1.778" layer="27" display="off"/>
 <attribute name="VALUE" x="7.296" y="26.162" size="1.016" layer="27" rot="R90" align="top-center"/>
 </element>
-<element name="C5" library="MyRCL" package="C0805" package3d_urn="urn:adsk.eagle:package:23617/2" value="4,7µF" x="9.906" y="29.083" smashed="yes">
+<element name="C5" library="MyRCL" package="C0805" package3d_urn="urn:adsk.eagle:package:23617/2" value="4.7uF" x="9.906" y="29.083" smashed="yes">
 <attribute name="NAME" x="8.101" y="29.083" size="1.016" layer="25" rot="R90" align="bottom-center"/>
 <attribute name="SPICEPREFIX" value="C" x="25.146" y="-30.607" size="1.778" layer="27" display="off"/>
@@
 <attribute name="VALUE" x="21.336" y="52.267" size="1.016" layer="27" align="top-center"/>
 </element>
-<element name="C18" library="MyRCL" package="C0805" package3d_urn="urn:adsk.eagle:package:23617/2" value="10µF" x="14.732" y="58.674" smashed="yes" rot="R270">
+<element name="C18" library="MyRCL" package="C0805" package3d_urn="urn:adsk.eagle:package:23617/2" value="10uF" x="14.732" y="58.674" smashed="yes" rot="R270">
 <attribute name="NAME" x="14.732" y="60.479" size="1.016" layer="25" align="bottom-center"/>
 <attribute name="SPICEPREFIX" value="C" x="5.842" y="63.754" size="1.778" layer="27" rot="R270" display="off"/>
